File: mga_expansion/mga_expansion.kicad_pcb (KiCad board)
At the start: 2 copper layers, 0 parts

Commit message: initial board outline and component placement
Parts:
- added J1: Bus_ISA_8bit, local:BUS_XT, F.Cu at (128.8, 135.2)
- added R1: 330, Resistor_THT:R_Axial_DIN0207_L6.3mm_D2.5mm_P10.16mm_Horizontal, F.Cu at (107.2, 115.1)
- added R2: 330, Resistor_THT:R_Axial_DIN0207_L6.3mm_D2.5mm_P10.16mm_Horizontal, F.Cu at (109.7, 115.1)
- added R3: 330, Resistor_THT:R_Axial_DIN0207_L6.3mm_D2.5mm_P10.16mm_Horizontal, F.Cu at (112.2, 115.1)
- added R4: 330, Resistor_THT:R_Axial_DIN0207_L6.3mm_D2.5mm_P10.16mm_Horizontal, F.Cu at (114.8, 115.1)
- added R5: 330, Resistor_THT:R_Axial_DIN0207_L6.3mm_D2.5mm_P10.16mm_Horizontal, F.Cu at (117.3, 115.1)
- added R6: 330, Resistor_THT:R_Axial_DIN0207_L6.3mm_D2.5mm_P10.16mm_Horizontal, F.Cu at (119.9, 115.1)
- added R7: 330, Resistor_THT:R_Axial_DIN0207_L6.3mm_D2.5mm_P10.16mm_Horizontal, F.Cu at (122.4, 115.1)
- added R8: 330, Resistor_THT:R_Axial_DIN0207_L6.3mm_D2.5mm_P10.16mm_Horizontal, F.Cu at (125.0, 115.1)
- added U1: W86855AF, Package_QFP:PQFP-100_14x20mm_P0.65mm, F.Cu at (94.4, 96.6)
Other:
- board outline added: 102.5 x 89.1 mm
